File: Hardware/master/Kirov_GPS/gps.sch (EAGLE design)
At the start: 7 parts

Commit message: added board layout and cap to schematic
Parts:
- added C1: 100 uf, SparkFun-Passives:CAPPTH1
Connections:
- net GND: now also C1.2
- net VCC: now also C1.1
Changed lines of the file:
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@@
 <part name="RX1JP" library="SparkFun-Connectors" deviceset="M03" device="LONGPADS"/>
 <part name="RX2JP" library="SparkFun-Connectors" deviceset="M03" device="LONGPADS"/>
+<part name="C1" library="SparkFun-Passives" deviceset="CAP" device="PTH1" value="100 uf"/>
 </parts>
 <sheets>
@@
 <instance part="RX1JP" gate="G$1" x="53.34" y="86.36" rot="R270"/>
 <instance part="RX2JP" gate="G$1" x="71.12" y="86.36" rot="R270"/>
+<instance part="C1" gate="G$1" x="48.26" y="58.42"/>
 </instances>
 <busses>
@@
 <wire x1="78.74" y1="66.04" x2="73.66" y2="66.04" width="0.1524" layer="91"/>
 <label x="73.66" y="66.04" size="1.778" layer="95"/>
+</segment>
+<segment>
+<pinref part="C1" gate="G$1" pin="1"/>
+<wire x1="48.26" y1="63.5" x2="48.26" y2="66.04" width="0.1524" layer="91"/>
+<label x="48.26" y="66.04" size="1.778" layer="95"/>
 </segment>
 </net>
@@
 <label x="73.66" y="63.5" size="1.778" layer="95"/>
 </segment>
+<segment>
+<pinref part="C1" gate="G$1" pin="2"/>
+<wire x1="48.26" y1="55.88" x2="48.26" y2="53.34" width="0.1524" layer="91"/>
+<label x="48.26" y="53.34" size="1.778" layer="95"/>
+</segment>
 </net>
